Commit message: Office tasks: ROS 2 bridge, SLAM, Nav2 and box pick-and-place; gait v14 policy
- deploy/isaac: office collision, ROS 2 interface (clock, odom, tf, joint
  states, head lidar, chest D435; /cmd_vel, arm poses, grippers), handle box,
  pickup table and grasping, sensor mounts from the vendor CAD
- ros2_ws: install and environment scripts for Humble, x1_bringup package with
  mapping and navigation launch files, Nav2 tuned to the walking policy,
  mapping route, map saver, fetch_box task node, and the saved office map
- manip: MuJoCo squeeze and handle-box studies
- policy: gait v14 (shoulder-width stance, softer knees, grippers, lidar and
  hand payload), Isaac URDF regenerated to match
- README: ROS 2 setup and run instructions, updated results

File: deploy/isaac/x1_isaac/x1_isaac.urdf (robot description, URDF)
Before this commit: robot agibot_x1_policy, 32 links, 31 joints
Links:
- added link left_gripper, mass 0.49
- added link mid360, mass 0.265
- added link right_gripper, mass 0.49
Joints:
- added joint left_gripper_fixed: type fixed, parent left_wrist_roll, child left_gripper, origin xyz=0 -0.09 0 rpy=0 -0 0
- added joint mid360_fixed: type fixed, parent torso_link, child mid360, origin xyz=0.0345 0.51 0 rpy=0 -0 0
- added joint right_gripper_fixed: type fixed, parent right_wrist_roll, child right_gripper, origin xyz=0 -0.09 0 rpy=0 -0 0
